File: schmatics/node3/node3.kicad_sch (KiCad schematic)
At the start: 0 parts

Commit message: Add Node 3 Schematic
Parts:
- added J1, J4: Conn_01x19, symbol Connector_Generic:Conn_01x19
- added MCP1: CAN Controller, symbol Connector_Generic:Conn_01x07
- added NEO-6M1: GPS Module, symbol Connector_Generic:Conn_01x04
- added Nextion2: Display, symbol Connector_Generic:Conn_01x04
Connections:
- new net: J4.1 (3V3), NEO-6M1.1 (VCC)
- new net: J4.10 (26), Nextion2.1 (RX)
- new net: J4.14 (GND), MCP1.6 (GND)
- new net: J4.15 (13), MCP1.2 (SCK)
- new net: J4.9 (25), Nextion2.2 (TX)
- new net: J1.7 (4), MCP1.1 (INT)
- new net: J1.18 (23), MCP1.3 (SI)
- new net: J1.12 (19), MCP1.4 (SO)
- new net: J1.10 (5), MCP1.5 (CS)
- new net: J1.13 (GND), Nextion2.3 (GND)
- new net: J1.19 (GND), NEO-6M1.2 (GND)
- new net: J1.8 (16), NEO-6M1.3 (TX)
- new net: J1.9 (17), NEO-6M1.4 (RX)
- new net +5V: J4.19 (5V), MCP1.7 (VCC), Nextion2.4 (+5V)
Other:
- company: (none) -> Triton Solar Car
- title: (none) -> Node 3: GPS & Dashboard
